Commit message: add gripper_joint to the URDF

File: test/test_resources/test_robot.urdf (robot description, URDF)
Before this commit: robot two_dof_robot, 13 links, 12 joints
Links:
- added link gripper_link, mass 0.002
Joints:
- added joint gripper_joint: type prismatic, parent gripper_left_finger, child gripper_link, origin xyz=0 0 0 rpy=0 0 0, axis 0 1 0, limit lower=-0.045 upper=0.045 effort=100 velocity=0.1
